Commit message: ✨feat:submoduleなど

File: urdf_test/urdf/agv3.urdf (robot description, URDF)
Before this commit: robot sam_bot, 11 links, 10 joints
Links:
- added link imu_link; visual box size=0.002 1.002 1; visual box size=0.015 0.011 0.012
Joints:
- added joint imu_joint: type fixed, parent base_link, child imu_link, origin xyz=0 0 1 rpy=0 0 0
